Commit message: added config file for bridging ros topics with gazebo,added world and map files, modified launch file to launch custom gazebo world and updated urdf file for adding 2d lidar

File: warehouse_robot/description/warehouse_bot.urdf (robot description, URDF)
Before this commit: robot warehouse_bot, 6 links, 5 joints
Links:
- link castor_wheel_link: mass 1.0 -> 0.5
